File: lna-filt.sch (KiCad schematic (older format))
At the start: 27 parts, among them J1 Conn_Coaxial, J2 Conn_Coaxial, J3 Barrel_Jack, J4 USB_B_Micro, J5 Conn_Coaxial, J6 Conn_Coaxial, U1 HMC374, U2 MCP1703A-3302_SOT223

Commit message: Move LED to 3V3, add power silk screen
Closes #2
Connections:
- net +3V3: now also R1.2
- net +5V: no longer R1.2
Changed lines of the file:
@@
-$EndComp
-$Comp
-L power:+5V #PWR0110
-U 1 1 5EB2F9D9
-P 6250 5350
-F 0 "#PWR0110" H 6250 5200 50  0001 C CNN
-F 1 "+5V" H 6265 5523 50  0000 C CNN
-F 2 "" H 6250 5350 50  0001 C CNN
-F 3 "" H 6250 5350 50  0001 C CNN
-	1    6250 5350
-	1    0    0    -1
 $EndComp
 $Comp
@@
 Wire Wire Line
 	7300 1250 7500 1250
+$Comp
+L power:+3V3 #PWR?
+U 1 1 5ECC153A
+P 6250 5350
+F 0 "#PWR?" H 6250 5200 50  0001 C CNN
+F 1 "+3V3" H 6265 5523 50  0000 C CNN
+F 2 "" H 6250 5350 50  0001 C CNN
+F 3 "" H 6250 5350 50  0001 C CNN
+	1    6250 5350
+	1    0    0    -1
+$EndComp
 $EndSCHEMATC
